Commit message: update pull and urdf

File: examples/assets/brackets.urdf (robot description, URDF)
Before this commit: robot onshnap, 12 links, 11 joints
Links:
- removed link link_Part_12_1
- removed link link_standoff1_1
- removed link link_standoff2_1
- removed link link_standoff3_1
- removed link link_standoff4_1
- removed link link_tower_first_tier_1
- added link link_Camera_1, mass 1.006291; collision mesh filename=meshes/Camera_1.stl; visual mesh filename=meshes/Camera_1.stl
- added link link_Camera_1_centroid, mass 0.000001
- added link link_Camera_2, mass 1.006291; collision mesh filename=meshes/Camera_2.stl; visual mesh filename=meshes/Camera_2.stl
- added link link_Camera_2_centroid, mass 0.000001
- added link link_Camera_3, mass 1.006291; collision mesh filename=meshes/Camera_3.stl; visual mesh filename=meshes/Camera_3.stl
- added link link_Camera_3_centroid, mass 0.000001
- added link link_Camera_4, mass 1.006291; collision mesh filename=meshes/Camera_4.stl; visual mesh filename=meshes/Camera_4.stl
- added link link_Camera_4_centroid, mass 0.000001
- added link link_back_high_bracket_1_centroid, mass 0.000001
- added link link_oak-d-pro_bracket_1_centroid, mass 0.000001
- added link link_oak-d-pro_bracket_2_centroid, mass 0.000001
- added link link_oak-d-pro_bracket_3_centroid, mass 0.000001
- added link link_tower_second_tier_1_centroid, mass 0.000001
- link link_back_high_bracket_1: mass 0.000000 -> 1.135597
- link link_oak-d-pro_bracket_1: mass 0.000000 -> 0.421565
- link link_oak-d-pro_bracket_2: mass 0.000000 -> 0.421565
- link link_oak-d-pro_bracket_3: mass 0.000000 -> 0.421565
- link link_tower_second_tier_1: mass 0.000000 -> 3.372220
Joints:
- removed joint joint_Part_12_1
- removed joint joint_standoff1_1
- removed joint joint_standoff2_1
- removed joint joint_standoff3_1
- removed joint joint_standoff4_1
- removed joint joint_tower_first_tier_1
- added joint joint_Camera_1: type fixed, parent base_link, child link_Camera_1, origin xyz=0.00021612 -0.04425000 0.05585680 rpy=1.57079633 -0.00000000 -3.14159265
- added joint joint_Camera_1_centroid: type fixed, parent base_link, child link_Camera_1_centroid, origin xyz=0.00021709 -0.04467888 0.05586718 rpy=1.57079633 -0.00000000 -3.14159265
- added joint joint_Camera_2: type fixed, parent base_link, child link_Camera_2, origin xyz=-0.09693626 0.01798650 0.05585680 rpy=1.57079633 -1.16937060 -3.14159265
- added joint joint_Camera_2_centroid: type fixed, parent base_link, child link_Camera_2_centroid, origin xyz=-0.09733066 0.01781804 0.05586718 rpy=1.57079633 -1.16937060 -3.14159265
- added joint joint_Camera_3: type fixed, parent base_link, child link_Camera_3, origin xyz=-0.00880096 0.06500000 0.18160680 rpy=0.00000000 0.00000000 3.14159265
- added joint joint_Camera_3_centroid: type fixed, parent base_link, child link_Camera_3_centroid, origin xyz=-0.00879999 0.06501037 0.18203568 rpy=0.00000000 0.00000000 3.14159265
- added joint joint_Camera_4: type fixed, parent base_link, child link_Camera_4, origin xyz=0.09946683 0.01829863 0.05585680 rpy=1.57079633 1.16937060 -3.14159265
- added joint joint_Camera_4_centroid: type fixed, parent base_link, child link_Camera_4_centroid, origin xyz=0.09986199 0.01813194 0.05586718 rpy=1.57079633 1.16937060 -3.14159265
- added joint joint_back_high_bracket_1_centroid: type fixed, parent base_link, child link_back_high_bracket_1_centroid, origin xyz=0.00119904 0.08795395 0.08756841 rpy=-0.00000000 0.00000000 0.00000000
- added joint joint_oak-d-pro_bracket_1_centroid: type fixed, parent base_link, child link_oak-d-pro_bracket_1_centroid, origin xyz=-0.09850150 0.01767963 0.03637125 rpy=-0.00000000 0.00000000 -2.74016693
- added joint joint_oak-d-pro_bracket_2_centroid: type fixed, parent base_link, child link_oak-d-pro_bracket_2_centroid, origin xyz=0.10089959 0.01767963 0.03637125 rpy=-0.00000000 0.00000000 -0.40142573
- added joint joint_oak-d-pro_bracket_3_centroid: type fixed, parent base_link, child link_oak-d-pro_bracket_3_centroid, origin xyz=0.00119904 -0.04581072 0.03637125 rpy=-0.00000000 0.00000000 -1.57079633
- added joint joint_tower_second_tier_1_centroid: type fixed, parent base_link, child link_tower_second_tier_1_centroid, origin xyz=0.00119904 0.01448281 0.01768180 rpy=-0.00000000 0.00000000 0.00000000
- joint joint_back_high_bracket_1: origin xyz=0.00119904 -0.00000000 -0.00184320 rpy=0.00000000 0.00000000 0.00000000 -> xyz=0.00119904 -0.00000000 -0.00184320 rpy=-0.00000000 0.00000000 0.00000000
- joint joint_oak-d-pro_bracket_1: origin xyz=-0.13126833 0.06623666 -0.00184320 rpy=0.00000000 0.00000000 -2.74016693 -> xyz=-0.13126833 0.06623666 -0.00184320 rpy=-0.00000000 0.00000000 -2.74016693
- joint joint_oak-d-pro_bracket_2: origin xyz=0.08873233 -0.03962140 -0.00184320 rpy=0.00000000 0.00000000 -0.40142573 -> xyz=0.08873233 -0.03962140 -0.00184320 rpy=-0.00000000 0.00000000 -0.40142573
- joint joint_oak-d-pro_bracket_3: origin xyz=-0.05630096 -0.05700000 -0.00184320 rpy=0.00000000 0.00000000 -1.57079633 -> xyz=-0.05630096 -0.05700000 -0.00184320 rpy=-0.00000000 0.00000000 -1.57079633
- joint joint_tower_second_tier_1: origin xyz=0.00119904 -0.00000000 -0.00184320 rpy=0.00000000 0.00000000 0.00000000 -> xyz=0.00119904 -0.00000000 -0.00184320 rpy=-0.00000000 0.00000000 0.00000000
